File: master/KiCAD-PCB/KiCAD-PCB.kicad_pcb (KiCad board)
At the start: 2 copper layers, 65.5 x 67.8 mm, 11 parts, among them J1 Conn_01x08_Pin

Commit message: 3D Files, PCB board, code update
Parts:
- LED1: renamed from D1; value LED -> LED1
- LED2: renamed from D2; value LED -> LED2
- LED3: renamed from D3; value LED -> LED3
- moved Joystick1 3.32 mm to (129.7, 73.1)
Connections:
- Joystick1 pad 2: GPIO27 -> GPIO35
- Joystick1 pad 3: GPIO14 -> GPIO34
Routing:
- net GPIO34: track 0.00 -> 23.3 mm
- net GPIO35: track 0.00 -> 16.5 mm
- net GPIO27: track 10.9 -> 0.00 mm
- net GPIO14: track 10.9 -> 0.00 mm
- net +3.3V: track 156.9 -> 157.5 mm
Other:
- board text added: "JOYSTICK"
- board text removed: "Joystick"
Changed lines of the file:
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@@
 			(layer "F.Fab")
 		)
+		(fp_text user "DISPLAY LCD"
+			(at 6.5 10.5 -90)
+			(unlocked yes)
+			(layer "B.SilkS")
+			(effects
+				(font
+					(size 1 1)
+					(thickness 0.1)
+				)
+				(justify left bottom mirror)
+			)
+		)
 		(fp_text user "${REFERENCE}"
 			(at 0 8.89 270)
@@
 		(descr "LED, diameter 5.0mm, 2 pins, http://cdn-reichelt.de/documents/datenblatt/A500/LL-504BC2E-009.pdf, generated by kicad-footprint-generator")
 		(tags "LED")
-		(property "Reference" "D3"
-			(at 1.5 -3.96 -0)
+		(property "Reference" "LED3"
+			(at 0.8 5.9 0)
 			(layer "B.SilkS")
 			(effects
@@
 			)
 		)
-		(property "Value" "LED"
-			(at 1.5 3.96 -0)
+		(property "Value" "LED3"
+			(at 1.5 3.96 0)
 			(layer "B.Fab")
 			(effects
@@
 		)
 		(property "Datasheet" ""
-			(at 2.77 0 -0)
+			(at 2.77 0 0)
 			(layer "B.Fab")
 			(hide yes)
@@
 		)
 		(property "Description" "Light emitting diode"
-			(at 2.77 0 -0)
+			(at 2.77 0 0)
 			(layer "B.Fab")
 			(hide yes)
@@
 		)
 		(property "Sim.Pins" "1=K 2=A"
-			(at 2.77 0 -0)
+			(at 2.77 0 0)
 			(unlocked yes)
 			(layer "B.Fab")
@@
 		)
 		(fp_text user "${REFERENCE}"
-			(at 1.5 0 -0)
+			(at 1.5 0 0)
 			(layer "B.Fab")
 			(effects
@@
 		(descr "LED, diameter 5.0mm, 2 pins, http://cdn-reichelt.de/documents/datenblatt/A500/LL-504BC2E-009.pdf, generated by kicad-footprint-generator")
 		(tags "LED")
-		(property "Reference" "D1"
-			(at 1.29 -3.96 -0)
+		(property "Reference" "LED1"
+			(at 1.3 8.1 0)
 			(layer "B.SilkS")
 			(effects
@@
 			)
 		)
-		(property "Value" "LED"
-			(at 1.29 3.96 -0)
+		(property "Value" "LED1"
+			(at 1.29 3.96 0)
 			(layer "B.Fab")
 			(effects
@@
 		)
 		(property "Datasheet" ""
-			(at 2.56 0 -0)
+			(at 2.56 0 0)
 			(layer "B.Fab")
 			(hide yes)
@@
 		)
 		(property "Description" "Light emitting diode"
-			(at 2.56 0 -0)
+			(at 2.56 0 0)
 			(layer "B.Fab")
 			(hide yes)
@@
 		)
 		(property "Sim.Pins" "1=K 2=A"
-			(at 2.56 0 -0)
+			(at 2.56 0 0)
 			(unlocked yes)
 			(layer "B.Fab")
@@
 		)
 		(fp_text user "${REFERENCE}"
-			(at 1.29 0 -0)
+			(at 1.29 0 0)
 			(layer "B.Fab")
 			(effects
@@
 	(footprint "Connector_PinSocket_2.54mm:PinSocket_1x05_P2.54mm_Vertical"
 		(layer "F.Cu")
-		(at 126.800001 71.509023 180)
+		(at 129.72 73.093736 180)
 		(descr "Through hole straight socket strip, 1x05, 2.54mm pitch, single row (from Kicad 4.0.7), script generated")
 		(tags "Through hole socket strip THT 1x05 2.54mm single row")
@@
 			(layers "*.Cu" "*.Mask")
 			(remove_unused_layers no)
-			(net 25 "GPIO27")
+			(net 22 "GPIO35")
 			(pinfunction "+5V")
 			(pintype "bidirectional")
@@
 			(layers "*.Cu" "*.Mask")
 			(remove_unused_layers no)
-			(net 26 "GPIO14")
+			(net 21 "GPIO34")
 			(pinfunction "VRX")
 			(pintype "bidirectional")
@@
 		(descr "LED, diameter 5.0mm, 2 pins, http://cdn-reichelt.de/documents/datenblatt/A500/LL-504BC2E-009.pdf, generated by kicad-footprint-generator")
 		(tags "LED")
-		(property "Reference" "D2"
-			(at 1.29 -3.96 -0)
+		(property "Reference" "LED2"
+			(at 0.9 8.2 0)
 			(layer "B.SilkS")
 			(effects
@@
 			)
 		)
-		(property "Value" "LED"
-			(at 1.29 3.96 -0)
+		(property "Value" "LED2"
+			(at 1.29 3.96 0)
 			(layer "B.Fab")
 			(effects
@@
 		)
 		(property "Datasheet" ""
-			(at 2.56 0 -0)
+			(at 2.56 0 0)
 			(layer "B.Fab")
 			(hide yes)
@@
 		)
 		(property "Description" "Light emitting diode"
-			(at 2.56 0 -0)
+			(at 2.56 0 0)
 			(layer "B.Fab")
 			(hide yes)
@@
 		)
 		(property "Sim.Pins" "1=K 2=A"
-			(at 2.56 0 -0)
+			(at 2.56 0 0)
 			(unlocked yes)
 			(layer "B.Fab")
@@
 		)
 		(fp_text user "${REFERENCE}"
-			(at 1.29 0 -0)
+			(at 1.29 0 0)
 			(layer "B.Fab")
 			(effects
@@
 		(at 148.570618 67.329023)
 		(property "Reference" "ESP32"
-			(at 6.029382 -28.229023 0)
+			(at 3.229382 31.470977 180)
 			(layer "B.SilkS")
 			(effects
@@
 		(layer "Edge.Cuts")
 	)
-	(gr_text "Joystick"
+	(gr_text "JOYSTICK"
 		(at 122.2 66.4 90)
 		(layer "B.SilkS")
@@
 	)
 	(segment
-		(start 126.800001 63.889023)
-		(end 127.840001 63.889023)
+		(start 132.800001 50.929023)
+		(end 132.800001 63.893735)
 		(width 1)
 		(layer "B.Cu")
@@
 	)
 	(segment
+		(start 132.800001 63.893735)
+		(end 131.22 65.473736)
+		(width 1)
+		(layer "B.Cu")
+		(net 8)
+	)
+	(segment
 		(start 177.300001 60.229023)
 		(end 172.500001 55.429023)
@@
 	)
 	(segment
-		(start 170.200001 39.629023)
-		(end 172.500001 41.929023)
+		(start 131.22 65.473736)
+		(end 129.72 65.473736)
 		(width 1)
 		(layer "B.Cu")
@@
 	)
 	(segment
-		(start 127.840001 63.889023)
-		(end 132.800001 58.929023)
+		(start 134.300001 49.429023)
+		(end 132.800001 50.929023)
 		(width 1)
 		(layer "B.Cu")
@@
 	)
 	(segment
-		(start 177.300001 62.3)
-		(end 174.6 62.3)
+		(start 159.100001 39.629023)
+		(end 149.300001 49.429023)
 		(width 1)
 		(layer "B.Cu")
@@
 	)
 	(segment
-		(start 149.300001 49.429023)
-		(end 159.100001 39.629023)
+		(start 177.300001 62.3)
+		(end 174.6 62.3)
 		(width 1)
 		(layer "B.Cu")
@@
 	)
 	(segment
-		(start 134.300001 49.429023)
-		(end 149.300001 49.429023)
+		(start 172.500001 41.929023)
+		(end 170.200001 39.629023)
 		(width 1)
 		(layer "B.Cu")
@@
 	)
 	(segment
-		(start 172.500001 41.929023)
-		(end 172.500001 55.429023)
+		(start 149.300001 49.429023)
+		(end 134.300001 49.429023)
 		(width 1)
 		(layer "B.Cu")
@@
 	)
 	(segment
-		(start 132.800001 58.929023)
-		(end 132.800001 50.929023)
-		(width 1)
-		(layer "B.Cu")
-		(net 8)
-	)
-	(segment
-		(start 159.100001 39.629023)
-		(end 170.200001 39.629023)
+		(start 170.200001 39.629023)
+		(end 159.100001 39.629023)
 		(width 1)
 		(layer "B.Cu")
@@
 	)
 	(segment
-		(start 132.800001 50.929023)
-		(end 134.300001 49.429023)
+		(start 172.500001 55.429023)
+		(end 172.500001 41.929023)
 		(width 1)
 		(layer "B.Cu")
@@
 	)
 	(segment
-		(start 138.305977 69.594023)
-		(end 140.700001 67.199999)
+		(start 125.2 70.5)
+		(end 125.2 76)
 		(width 1)
 		(layer "B.Cu")
-		(net 23)
+		(net 21)
 	)
 	(segment
-		(start 135.870618 69.594023)
-		(end 138.305977 69.594023)
+		(start 128.954023 79.754023)
+		(end 135.870618 79.754023)
 		(width 1)
 		(layer "B.Cu")
-		(net 23)
+		(net 21)
 	)
 	(segment
-		(start 140.700001 67.199999)
-		(end 140.700001 56.889023)
+		(start 129.72 68.013736)
+		(end 127.686264 68.013736)
 		(width 1)
 		(layer "B.Cu")
-		(net 23)
+		(net 21)
 	)
 	(segment
-		(start 126.800001 71.509023)
-		(end 129.490977 71.509023)
+		(start 127.686264 68.013736)
+		(end 125.2 70.5)
 		(width 1)
 		(layer "B.Cu")
-		(net 24)
+		(net 21)
 	)
 	(segment
-		(start 129.490977 71.509023)
-		(end 133.945977 67.054023)
+		(start 125.2 76)
+		(end 128.954023 79.754023)
 		(width 1)
 		(layer "B.Cu")
-		(net 24)
+		(net 21)
 	)
 	(segment
-		(start 133.945977 67.054023)
-		(end 135.870618 67.054023)
+		(start 129.72 70.553736)
+		(end 127.646264 70.553736)
 		(width 1)
 		(layer "B.Cu")
-		(net 24)
+		(net 22)
 	)
 	(segment
-		(start 135.870618 64.514023)
-		(end 133.215001 64.514023)
+		(start 127 74.9)
+		(end 129.314023 77.214023)
 		(width 1)
 		(layer "B.Cu")
-		(net 25)
+		(net 22)
 	)
 	(segment
-		(start 128.760001 68.969023)
-		(end 126.800001 68.969023)
+		(start 127.646264 70.553736)
+		(end 127 71.2)
 		(width 1)
 		(layer "B.Cu")
-		(net 25)
+		(net 22)
 	)
 	(segment
-		(start 133.215001 64.514023)
-		(end 128.760001 68.969023)
+		(start 127 71.2)
+		(end 127 74.9)
 		(width 1)
 		(layer "B.Cu")
-		(net 25)
+		(net 22)
 	)
 	(segment
-		(start 126.800001 66.429023)
-		(end 128.300001 66.429023)
+		(start 129.314023 77.214023)
+		(end 135.870618 77.214023)
 		(width 1)
 		(layer "B.Cu")
-		(net 26)
+		(net 22)
 	)
 	(segment
-		(start 132.755001 61.974023)
-		(end 135.870618 61.974023)
+		(start 138.305977 69.594023)
+		(end 140.700001 67.199999)
 		(width 1)
 		(layer "B.Cu")
-		(net 26)
+		(net 23)
 	)
 	(segment
-		(start 128.300001 66.429023)
-		(end 132.755001 61.974023)
+		(start 135.870618 69.594023)
+		(end 138.305977 69.594023)
 		(width 1)
 		(layer "B.Cu")
-		(net 26)
+		(net 23)
+	)
+	(segment
+		(start 140.700001 67.199999)
+		(end 140.700001 56.889023)
+		(width 1)
+		(layer "B.Cu")
+		(net 23)
+	)
+	(segment
+		(start 131.806264 73.093736)
+		(end 129.72 73.093736)
+		(width 1)
+		(layer "B.Cu")
+		(net 24)
+	)
+	(segment
+		(start 132.8 68.2)
+		(end 132.8 72.1)
+		(width 1)
+		(layer "B.Cu")
+		(net 24)
+	)
+	(segment
+		(start 133.945977 67.054023)
+		(end 132.8 68.2)
+		(width 1)
+		(layer "B.Cu")
+		(net 24)
+	)
+	(segment
+		(start 132.8 72.1)
+		(end 131.806264 73.093736)
+		(width 1)
+		(layer "B.Cu")
+		(net 24)
+	)
+	(segment
+		(start 133.945977 67.054023)
+		(end 135.870618 67.054023)
+		(width 1)
+		(layer "B.Cu")
+		(net 24)
 	)
 	(segment
