File: master/KiCAD-PCB/KiCAD-PCB.kicad_sch (KiCad schematic)
At the start: 11 parts, among them J1 Conn_01x08_Pin

Commit message: 3D Files, PCB board, code update
Parts:
- renumbered 220Ohm to 220Ohm1, 220Ohm to 220Ohm2, 220Ohm to 220Ohm3
Connections:
- net GPIO26: no longer Joystick1.3 (VRX)
- net GPIO27: no longer Joystick1.4 (VRY)
- net GPIO34: now also Joystick1.3 (VRX)
- net GPIO35: now also Joystick1.4 (VRY)
Changed lines of the file:
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@@
+		)
+	)
+	(global_label "GPIO35"
+		(shape input)
+		(at 27.94 113.03 180)
+		(fields_autoplaced yes)
+		(effects
+			(font
+				(size 1.27 1.27)
+			)
+			(justify right)
+		)
+		(property "Intersheetrefs" "${INTERSHEET_REFS}"
+			(at 18.0605 113.03 0)
+			(effects
+				(font
+					(size 1.27 1.27)
+				)
+				(justify right)
+				(hide yes)
+			)
 		)
 	)
@@
 		)
 	)
+	(global_label "GPIO34"
+		(shape input)
+		(at 27.94 110.49 180)
+		(fields_autoplaced yes)
+		(effects
+			(font
+				(size 1.27 1.27)
+			)
+			(justify right)
+		)
+		(property "Intersheetrefs" "${INTERSHEET_REFS}"
+			(at 18.0605 110.49 0)
+			(effects
+				(font
+					(size 1.27 1.27)
+				)
+				(justify right)
+				(hide yes)
+			)
+		)
+	)
 	(global_label "GPIO25"
 		(shape input)
@@
 		)
 	)
-	(global_label "GPIO26"
-		(shape input)
-		(at 27.94 110.49 180)
+	(global_label "GPIO23"
+		(shape input)
+		(at 93.98 111.76 0)
+		(fields_autoplaced yes)
+		(effects
+			(font
+				(size 1.27 1.27)
+			)
+			(justify left)
+		)
+		(property "Intersheetrefs" "${INTERSHEET_REFS}"
+			(at 103.8595 111.76 0)
+			(effects
+				(font
+					(size 1.27 1.27)
+				)
+				(justify left)
+				(hide yes)
+			)
+		)
+	)
+	(global_label "GPIO23"
+		(shape input)
+		(at 92.71 55.88 180)
 		(fields_autoplaced yes)
 		(effects
@@
 		)
 		(property "Intersheetrefs" "${INTERSHEET_REFS}"
-			(at 18.0605 110.49 0)
+			(at 82.8305 55.88 0)
 			(effects
 				(font
@@
 	(global_label "GPIO23"
 		(shape input)
-		(at 93.98 111.76 0)
+		(at 60.96 40.005 0)
 		(fields_autoplaced yes)
 		(effects
@@
 		)
 		(property "Intersheetrefs" "${INTERSHEET_REFS}"
-			(at 103.8595 111.76 0)
-			(effects
-				(font
-					(size 1.27 1.27)
-				)
-				(justify left)
-				(hide yes)
-			)
-		)
-	)
-	(global_label "GPIO23"
-		(shape input)
-		(at 92.71 55.88 180)
-		(fields_autoplaced yes)
-		(effects
-			(font
-				(size 1.27 1.27)
-			)
-			(justify right)
-		)
-		(property "Intersheetrefs" "${INTERSHEET_REFS}"
-			(at 82.8305 55.88 0)
-			(effects
-				(font
-					(size 1.27 1.27)
-				)
-				(justify right)
-				(hide yes)
-			)
-		)
-	)
-	(global_label "GPIO23"
-		(shape input)
-		(at 60.96 40.005 0)
-		(fields_autoplaced yes)
-		(effects
-			(font
-				(size 1.27 1.27)
-			)
-			(justify left)
-		)
-		(property "Intersheetrefs" "${INTERSHEET_REFS}"
 			(at 70.8395 40.005 0)
 			(effects
@@
 				)
 				(justify left)
-				(hide yes)
-			)
-		)
-	)
-	(global_label "GPIO27"
-		(shape input)
-		(at 27.94 113.03 180)
-		(fields_autoplaced yes)
-		(effects
-			(font
-				(size 1.27 1.27)
-			)
-			(justify right)
-		)
-		(property "Intersheetrefs" "${INTERSHEET_REFS}"
-			(at 18.0605 113.03 0)
-			(effects
-				(font
-					(size 1.27 1.27)
-				)
-				(justify right)
 				(hide yes)
 			)
@@
 		(on_board yes)
 		(dnp no)
-		(property "Reference" "220Ohm"
+		(property "Reference" "220Ohm2"
 			(at 146.304 110.998 90)
 			(effects
@@
 			(project "IC_GabrielVictor"
 				(path "/6989ec71-7bb6-4043-be66-284884750dd3"
-					(reference "220Ohm")
+					(reference "220Ohm2")
 					(unit 1)
 				)
@@
 		(on_board yes)
 		(dnp no)
-		(property "Reference" "220Ohm"
+		(property "Reference" "220Ohm1"
 			(at 146.304 100.33 90)
 			(effects
@@
 			(project "IC_GabrielVictor"
 				(path "/6989ec71-7bb6-4043-be66-284884750dd3"
-					(reference "220Ohm")
+					(reference "220Ohm1")
 					(unit 1)
 				)
@@
 		(on_board yes)
 		(dnp no)
-		(property "Reference" "220Ohm"
+		(property "Reference" "220Ohm3"
 			(at 146.05 121.158 90)
 			(effects
@@
 			(project "IC_GabrielVictor"
 				(path "/6989ec71-7bb6-4043-be66-284884750dd3"
-					(reference "220Ohm")
+					(reference "220Ohm3")
 					(unit 1)
 				)
